File: kicad/kerstboom.kicad_sch (KiCad schematic)
At the start: 46 parts, among them J1 Serial, J2 I2C, J3 AD12, J4 AD34, J5 SPI-BUS, J6 NEOPixel, U1 XIAO, U2 VEML7700-TR

Commit message: fixed symbol lib misc cleanups kikad directory and PCB
Parts:
- C1, C2, C3, C4, C5: footprint OPL_Capacitor:C0805 -> Capacitor_SMD:C_0805_2012Metric
- H1, H2, H3, H4: footprint XIAO:MountingHole_3.2mm_M3 -> MountingHole:MountingHole_3.2mm_M3
- J1, J2, J3, J4: footprint OPL_Connector:GROVE-HW4-2.0-90D -> custom:GROVE-HW4-2.0-90D
- J6: value NEOPixel -> NeoPixel
- U1: footprint XIAO:Seeeduino XIAO-MOUDLE14P-2.54-21X17.8MM-holes -> custom:Seeeduino XIAO-MOUDLE14P-2.54-21X17.8MM-holes
- U2: footprint VEML7700:XDCR_VEML7700-TR -> custom:XDCR_VEML7700-TR
Connections:
- net +3.3V: now also R2.2; no longer R2.1
- net SDA: now also R2.1; no longer R2.2
Other:
- company: (none) -> Sensemakers/In2Tech
- title: (none) -> NeoPixel4Xiao
- moved on the sheet: C1, C3, C4, C5, H1, H3, H4, H5, H7, H8, H9, J6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
